File: Electronic Load/Electronic Load.sch (KiCad schematic (older format))
At the start: 12 parts

Commit message: Updated Schematics
Parts:
- removed R?: 1k, symbol Device:R
- removed R? (x3): 5k Trim, symbol Device:RTRIM
- removed RV?: Current Level, symbol Device:R_POT
- removed SW?: SW_DIP_x01, symbol Switch:SW_DIP_x01
- added D?: Red, symbol Device:LED
- added R? (x2): R, symbol Device:R
- added R? (x2): 10k, symbol Device:R
- added R?: 220, symbol Device:R
- added SW?: Rotary_Encoder_Switch, symbol Device:Rotary_Encoder_Switch
- added U?: MCP4551, symbol Electronic~Load:MCP4551
- added U?: ATtiny84-20SSU, Package_SO:SOIC-14_3.9x8.7mm_P1.27mm, symbol MCU_Microchip_ATtiny:ATtiny84-20SSU
- added U?: SSD1306, symbol Electronic~Load:SSD1306
Connections:
- net labels added: EncA, EncB, Enc_SW, MISO, RESET, SCL, SDA_MOSI
- wire segments 38 -> 67

Commit message: Updated Schematics
Parts:
- removed J?: Load In, symbol Connector_Generic:Conn_01x02
- removed J?: 5V Power, symbol Connector_Generic:Conn_01x02
- added C1, C2: 0.01uF, symbol Device:C
- added J1: Load_IN, symbol Connector_Generic:Conn_01x01
- added J3: Programming Header, symbol Connector_Generic:Conn_01x05
- added J4: Load_OUT, symbol Connector_Generic:Conn_01x01
- added M2, M3: MNMOS, symbol pspice:MNMOS
- added P1: USB_C_Plug_USB2.0, symbol Connector:USB_C_Plug_USB2.0
- added R6, R7: 10k, symbol Device:R
- gave numbers to parts that had none: 13
Connections:
- net labels added: Gate
- wire segments 67 -> 101
Other:
- moved on the sheet: R1, R2, SW1

Commit message: Updated Schematic
Parts:
- removed P1: USB_C_Plug_USB2.0, symbol Connector:USB_C_Plug_USB2.0
- added J2: Fan Connector, Connector_Harwin:Harwin_LTek-Male_02_P2.00mm_Vertical, symbol Connector_Generic:Conn_01x02
- added J5: USB_C_Receptacle, Connector_USB:USB_C_Receptacle_Amphenol_12401610E4-2A, symbol Connector:USB_C_Receptacle
- added M4: MNMOS, Package_TO_SOT_SMD:TO-263-2, symbol pspice:MNMOS
- added R8: 10k, Resistor_SMD:R_1206_3216Metric, symbol Device:R
- added TH1: 10k, Diode_SMD:D_SOD-523, symbol Device:Thermistor_PTC
- C1, C2: footprint (none) -> Capacitor_SMD:C_1206_3216Metric
- D1: footprint (none) -> LED_SMD:LED_1206_3216Metric
- J1, J4: footprint (none) -> TerminalBlock_Wuerth:Wuerth_REDCUBE-THR_WP-THRBU_74650195_THR
- J3: footprint (none) -> Connector_Molex:Molex_KK-254_AE-6410-05A_1x05_P2.54mm_Vertical
- M1, M2, M3: footprint (none) -> Package_TO_SOT_SMD:TO-263-2
- R1, R2, R3, R4, R5, R6, R7: footprint (none) -> Resistor_SMD:R_1206_3216Metric
- SW1: footprint (none) -> Rotary_Encoder:RotaryEncoder_Alps_EC12E-Switch_Vertical_H20mm
- U2: footprint (none) -> Package_SO:MSOP-8-1EP_3x3mm_P0.65mm_EP1.95x2.15mm
- U4: footprint (none) -> Package_SON:Texas_S-PVSON-N8
Connections:
- net labels added: Fan_Pin, Tout
- wire segments 101 -> 117
Other:
- moved on the sheet: U4C

Commit message: Started PCB Layout
Parts:
- removed M1, M2, M3, M4: MNMOS, Package_TO_SOT_SMD:TO-263-2, symbol pspice:MNMOS
- added Q1, Q2, Q3, Q4: IRFS3306, Package_TO_SOT_SMD:TO-263-2, symbol Transistor_FET:IRFS4115
- U3: footprint (none) -> OLED:SSD1306_OLED
Connections:
- wire segments 117 -> 107
- no-connect marks 0 -> 1
Other:
- moved on the sheet: J5
Changed lines of the file:
@@
 $EndDescr
-$Comp
-L pspice:MNMOS M1
-U 1 1 610F10CA
-P 7550 3550
-F 0 "M1" H 7500 3800 50  0000 L CNN
-F 1 "MNMOS" H 7300 3700 50  0000 L CNN
-F 2 "Package_TO_SOT_SMD:TO-263-2" H 7525 3550 50  0001 C CNN
-F 3 "~" H 7525 3550 50  0001 C CNN
-	1    7550 3550
-	1    0    0    -1
-$EndComp
 $Comp
 L Sensor_Current:ACS758xCB-150U-PFF U5
@@
 Wire Wire Line
 	7650 3750 7650 3850
-Wire Wire Line
-	7750 3750 7750 3850
-Wire Wire Line
-	7750 3850 7650 3850
 Connection ~ 7650 3850
 Wire Wire Line
@@
 L power:GND #PWR018
 U 1 1 610F9C63
-P 9950 3550
-F 0 "#PWR018" H 9950 3300 50  0001 C CNN
-F 1 "GND" H 9955 3377 50  0000 C CNN
-F 2 "" H 9950 3550 50  0001 C CNN
-F 3 "" H 9950 3550 50  0001 C CNN
-	1    9950 3550
+P 10350 3550
+F 0 "#PWR018" H 10350 3300 50  0001 C CNN
+F 1 "GND" H 10355 3377 50  0000 C CNN
+F 2 "" H 10350 3550 50  0001 C CNN
+F 3 "" H 10350 3550 50  0001 C CNN
+	1    10350 3550
 	1    0    0    -1
 $EndComp
@@
 L power:+5V #PWR017
 U 1 1 610FA16B
-P 10650 750
-F 0 "#PWR017" H 10650 600 50  0001 C CNN
-F 1 "+5V" H 10665 923 50  0000 C CNN
-F 2 "" H 10650 750 50  0001 C CNN
-F 3 "" H 10650 750 50  0001 C CNN
-	1    10650 750
+P 11050 750
+F 0 "#PWR017" H 11050 600 50  0001 C CNN
+F 1 "+5V" H 11065 923 50  0000 C CNN
+F 2 "" H 11050 750 50  0001 C CNN
+F 3 "" H 11050 750 50  0001 C CNN
+	1    11050 750
 	1    0    0    -1
 $EndComp
@@
 	7450 3850 7650 3850
 Wire Wire Line
-	10550 850  10650 850
-Wire Wire Line
-	10650 850  10650 750
-Wire Wire Line
-	9950 3450 9950 3500
+	10950 850  11050 850
+Wire Wire Line
+	11050 850  11050 750
+Wire Wire Line
+	10350 3450 10350 3500
 Text Notes 6300 2650 0    50   ~ 0
 26.7mV/A
@@
 L power:GND #PWR06
 U 1 1 61141B6B
-P 2100 4550
-F 0 "#PWR06" H 2100 4300 50  0001 C CNN
-F 1 "GND" H 2105 4377 50  0000 C CNN
-F 2 "" H 2100 4550 50  0001 C CNN
-F 3 "" H 2100 4550 50  0001 C CNN
-	1    2100 4550
-	1    0    0    -1
-$EndComp
-Text GLabel 2100 4300 2    50   Input ~ 0
+P 2100 4300
+F 0 "#PWR06" H 2100 4050 50  0001 C CNN
+F 1 "GND" H 2105 4127 50  0000 C CNN
+F 2 "" H 2100 4300 50  0001 C CNN
+F 3 "" H 2100 4300 50  0001 C CNN
+	1    2100 4300
+	0    -1   -1   0
+$EndComp
+Text GLabel 2100 4500 2    50   Input ~ 0
 Enc_SW
 Wire Wire Line
@@
 Wire Wire Line
 	2000 4500 2100 4500
-Wire Wire Line
-	2100 4500 2100 4550
 Text GLabel 2050 1550 2    50   Input ~ 0
 MISO
@@
 F 0 "U3" H 4428 76  50  0000 L CNN
 F 1 "SSD1306" H 4428 -15 50  0000 L CNN
-F 2 "" H 4200 500 50  0001 C CNN
+F 2 "OLED:SSD1306_OLED" H 4200 500 50  0001 C CNN
 F 3 "" H 4200 500 50  0001 C CNN
 	1    4200 500
@@
 $EndComp
 Wire Wire Line
-	9650 3450 9650 3500
-Wire Wire Line
-	9650 3500 9950 3500
-Connection ~ 9950 3500
-Wire Wire Line
-	9950 3500 9950 3550
+	10050 3500 10350 3500
+Connection ~ 10350 3500
+Wire Wire Line
+	10350 3500 10350 3550
 $Comp
 L Device:R R6
@@
 Wire Wire Line
 	1100 4550 1350 4550
-$Comp
-L pspice:MNMOS M2
-U 1 1 611B1018
-P 8250 3550
-F 0 "M2" H 8200 3800 50  0000 L CNN
-F 1 "MNMOS" H 8000 3700 50  0000 L CNN
-F 2 "Package_TO_SOT_SMD:TO-263-2" H 8225 3550 50  0001 C CNN
-F 3 "~" H 8225 3550 50  0001 C CNN
-	1    8250 3550
-	1    0    0    -1
-$EndComp
-$Comp
-L pspice:MNMOS M3
-U 1 1 611B1745
-P 9100 3500
-F 0 "M3" H 9050 3750 50  0000 L CNN
-F 1 "MNMOS" H 8850 3650 50  0000 L CNN
-F 2 "Package_TO_SOT_SMD:TO-263-2" H 9075 3500 50  0001 C CNN
-F 3 "~" H 9075 3500 50  0001 C CNN
-	1    9100 3500
-	1    0    0    -1
-$EndComp
 Text GLabel 7150 3600 3    50   Input ~ 0
 Gate
 Text GLabel 8850 3550 3    50   Input ~ 0
 Gate
-Text GLabel 8000 3600 3    50   Input ~ 0
+Text GLabel 8100 3600 3    50   Input ~ 0
 Gate
 Wire Wire Line
-	8900 3500 8850 3500
-Wire Wire Line
 	8850 3500 8850 3550
-Wire Wire Line
-	8050 3550 8000 3550
-Wire Wire Line
-	8000 3550 8000 3600
 Wire Wire Line
 	7150 3600 7150 3550
@@
 Wire Wire Line
 	7150 3550 7350 3550
-Wire Wire Line
-	8350 3350 8350 3200
-Wire Wire Line
-	8350 3200 7650 3200
 Connection ~ 7650 3200
 Wire Wire Line
@@
 	9200 3300 9200 3200
 Wire Wire Line
-	9200 3200 8350 3200
-Connection ~ 8350 3200
-Wire Wire Line
-	8350 3750 8350 3850
-Wire Wire Line
-	8350 3850 7750 3850
-Connection ~ 7750 3850
-Wire Wire Line
-	8450 3750 8450 3850
-Wire Wire Line
-	8450 3850 8350 3850
-Connection ~ 8350 3850
-Wire Wire Line
 	9200 3700 9200 3850
-Connection ~ 8450 3850
-Wire Wire Line
-	9300 3700 9300 3850
-Wire Wire Line
-	8450 3850 9200 3850
-Connection ~ 9200 3850
-Wire Wire Line
-	9200 3850 9300 3850
 $Comp
 L Connector_Generic:Conn_01x02 J2
@@
 $EndComp
 $Comp
-L pspice:MNMOS M4
-U 1 1 6116A848
-P 10050 5200
-F 0 "M4" H 10000 5450 50  0000 L CNN
-F 1 "MNMOS" H 9800 5350 50  0000 L CNN
-F 2 "Package_TO_SOT_SMD:TO-263-2" H 10025 5200 50  0001 C CNN
-F 3 "~" H 10025 5200 50  0001 C CNN
-	1    10050 5200
-	1    0    0    -1
-$EndComp
-$Comp
 L power:+5V #PWR025
 U 1 1 6116BE08
@@
 $EndComp
 Wire Wire Line
-	10150 5400 10150 5450
-Wire Wire Line
-	10250 5400 10250 5450
-Wire Wire Line
-	10250 5450 10150 5450
-Connection ~ 10150 5450
-Wire Wire Line
-	10150 5450 10150 5500
-Wire Wire Line
 	10150 4700 10150 4800
 Wire Wire Line
@@
 L Connector:USB_C_Receptacle J5
 U 1 1 611AF3FF
-P 9950 1850
-F 0 "J5" H 10057 3117 50  0000 C CNN
-F 1 "USB_C_Receptacle" H 10057 3026 50  0000 C CNN
-F 2 "Connector_USB:USB_C_Receptacle_Amphenol_12401610E4-2A" H 10100 1850 50  0001 C CNN
-F 3 "https://www.usb.org/sites/default/files/documents/usb_type-c.zip" H 10100 1850 50  0001 C CNN
-	1    9950 1850
-	1    0    0    -1
-$EndComp
+P 10350 1850
+F 0 "J5" H 10457 3117 50  0000 C CNN
+F 1 "USB_C_Receptacle" H 10457 3026 50  0000 C CNN
+F 2 "Connector_USB:USB_C_Receptacle_Amphenol_12401610E4-2A" H 10500 1850 50  0001 C CNN
+F 3 "https://www.usb.org/sites/default/files/documents/usb_type-c.zip" H 10500 1850 50  0001 C CNN
+	1    10350 1850
+	1    0    0    -1
+$EndComp
+NoConn ~ 1950 2050
+$Comp
+L Transistor_FET:IRFS4115 Q4
+U 1 1 611744E8
+P 10050 5200
+F 0 "Q4" H 10255 5246 50  0000 L CNN
+F 1 "IRFS3306" H 10255 5155 50  0000 L CNN
+F 2 "Package_TO_SOT_SMD:TO-263-2" H 10250 5125 50  0001 L CIN
+F 3 "https://www.infineon.com/dgdl/irfs4115pbf.pdf?fileId=5546d462533600a401535636e5d2218f" H 10050 5200 50  0001 L CNN
+	1    10050 5200
+	1    0    0    -1
+$EndComp
+Wire Wire Line
+	10150 5400 10150 5500
+$Comp
+L Transistor_FET:IRFS4115 Q1
+U 1 1 611758CE
+P 7550 3550
+F 0 "Q1" H 7755 3596 50  0000 L CNN
+F 1 "IRFS3306" H 7650 3400 50  0000 L CNN
+F 2 "Package_TO_SOT_SMD:TO-263-2" H 7750 3475 50  0001 L CIN
+F 3 "https://www.infineon.com/dgdl/irfs4115pbf.pdf?fileId=5546d462533600a401535636e5d2218f" H 7550 3550 50  0001 L CNN
+	1    7550 3550
+	1    0    0    -1
+$EndComp
+$Comp
+L Transistor_FET:IRFS4115 Q2
+U 1 1 61178B60
+P 8350 3550
+F 0 "Q2" H 8555 3596 50  0000 L CNN
+F 1 "IRFS3306" H 8450 3400 50  0000 L CNN
+F 2 "Package_TO_SOT_SMD:TO-263-2" H 8550 3475 50  0001 L CIN
+F 3 "https://www.infineon.com/dgdl/irfs4115pbf.pdf?fileId=5546d462533600a401535636e5d2218f" H 8350 3550 50  0001 L CNN
+	1    8350 3550
+	1    0    0    -1
+$EndComp
+$Comp
+L Transistor_FET:IRFS4115 Q3
+U 1 1 61179166
+P 9100 3500
+F 0 "Q3" H 9305 3546 50  0000 L CNN
+F 1 "IRFS3306" H 9305 3455 50  0000 L CNN
+F 2 "Package_TO_SOT_SMD:TO-263-2" H 9300 3425 50  0001 L CIN
+F 3 "https://www.infineon.com/dgdl/irfs4115pbf.pdf?fileId=5546d462533600a401535636e5d2218f" H 9100 3500 50  0001 L CNN
+	1    9100 3500
+	1    0    0    -1
+$EndComp
+Wire Wire Line
+	8150 3550 8100 3550
+Wire Wire Line
+	8100 3550 8100 3600
+Wire Wire Line
+	7650 3850 8450 3850
+Wire Wire Line
+	7650 3200 8450 3200
+Wire Wire Line
+	8450 3350 8450 3200
+Connection ~ 8450 3200
+Wire Wire Line
+	8450 3200 9200 3200
+Wire Wire Line
+	8450 3750 8450 3850
+Connection ~ 8450 3850
+Wire Wire Line
+	8450 3850 9200 3850
+Wire Wire Line
+	8850 3500 8900 3500
+Wire Wire Line
+	10050 3450 10050 3500
 $EndSCHEMATC

Commit message: Updated PCB
Parts:
- added NT1: Net-Tie_2, NetTie:NetTie-2_SMD_Pad2.0mm, symbol Device:Net-Tie_2
Connections:
- wire segments 107 -> 110
Changed lines of the file:
@@
 L power:GND #PWR016
 U 1 1 610FC0E8
-P 7450 4000
-F 0 "#PWR016" H 7450 3750 50  0001 C CNN
-F 1 "GND" H 7455 3827 50  0000 C CNN
-F 2 "" H 7450 4000 50  0001 C CNN
-F 3 "" H 7450 4000 50  0001 C CNN
-	1    7450 4000
-	1    0    0    -1
-$EndComp
-Wire Wire Line
-	7450 3850 7650 3850
+P 7100 4100
+F 0 "#PWR016" H 7100 3850 50  0001 C CNN
+F 1 "GND" H 7105 3927 50  0000 C CNN
+F 2 "" H 7100 4100 50  0001 C CNN
+F 3 "" H 7100 4100 50  0001 C CNN
+	1    7100 4100
+	1    0    0    -1
+$EndComp
 Wire Wire Line
 	10950 850  11050 850
@@
 	1    0    0    -1
 $EndComp
-Wire Wire Line
-	7450 3850 7450 4000
 Wire Wire Line
 	5750 3550 7150 3550
@@
 Wire Wire Line
 	1000 7050 950  7050
+Text GLabel 1050 7150 2    50   Input ~ 0
+SDA_MOSI
 Text GLabel 1050 7250 2    50   Input ~ 0
-SDA_MOSI
-Text GLabel 1050 7150 2    50   Input ~ 0
 RESET
+Text GLabel 1050 7450 2    50   Input ~ 0
+MISO
 Text GLabel 1050 7350 2    50   Input ~ 0
-MISO
-Text GLabel 1050 7450 2    50   Input ~ 0
 SCL
 Wire Wire Line
@@
 Wire Wire Line
 	9750 5200 9850 5200
-Text GLabel 2050 2150 2    50   Input ~ 0
+Text GLabel 2050 2050 2    50   Input ~ 0
 Fan_Pin
-Wire Wire Line
-	1950 2150 2050 2150
 $Comp
 L Device:Thermistor_PTC TH1
@@
 	1    0    0    -1
 $EndComp
-NoConn ~ 1950 2050
 $Comp
 L Transistor_FET:IRFS4115 Q4
@@
 Wire Wire Line
 	10050 3450 10050 3500
+$Comp
+L Device:Net-Tie_2 NT1
+U 1 1 61171D25
+P 7350 4000
+F 0 "NT1" H 7350 4181 50  0000 C CNN
+F 1 "Net-Tie_2" H 7350 4090 50  0000 C CNN
+F 2 "NetTie:NetTie-2_SMD_Pad2.0mm" H 7350 4000 50  0001 C CNN
+F 3 "~" H 7350 4000 50  0001 C CNN
+	1    7350 4000
+	1    0    0    -1
+$EndComp
+Wire Wire Line
+	7450 4000 7550 4000
+Wire Wire Line
+	7550 4000 7550 3850
+Wire Wire Line
+	7550 3850 7650 3850
+Wire Wire Line
+	7250 4000 7100 4000
+Wire Wire Line
+	7100 4000 7100 4100
+Wire Wire Line
+	1950 2050 2050 2050
+NoConn ~ 1950 2150
 $EndSCHEMATC

Commit message: Updated PCB
Parts:
- added C3: 10uF, Capacitor_SMD:CP_Elec_4x5.4, symbol Device:C
Connections:
- wire segments 110 -> 112
Changed lines of the file:
@@
 	1950 2050 2050 2050
 NoConn ~ 1950 2150
+$Comp
+L Device:C C3
+U 1 1 611AD2AB
+P 9100 1050
+F 0 "C3" H 9215 1096 50  0000 L CNN
+F 1 "10uF" H 9215 1005 50  0000 L CNN
+F 2 "Capacitor_SMD:CP_Elec_4x5.4" H 9138 900 50  0001 C CNN
+F 3 "~" H 9100 1050 50  0001 C CNN
+	1    9100 1050
+	1    0    0    -1
+$EndComp
+$Comp
+L power:+5V #PWR0101
+U 1 1 611AD734
+P 9100 800
+F 0 "#PWR0101" H 9100 650 50  0001 C CNN
+F 1 "+5V" H 9115 973 50  0000 C CNN
+F 2 "" H 9100 800 50  0001 C CNN
+F 3 "" H 9100 800 50  0001 C CNN
+	1    9100 800
+	1    0    0    -1
+$EndComp
+$Comp
+L power:GND #PWR0102
+U 1 1 611ADC55
+P 9100 1300
+F 0 "#PWR0102" H 9100 1050 50  0001 C CNN
+F 1 "GND" H 9105 1127 50  0000 C CNN
+F 2 "" H 9100 1300 50  0001 C CNN
+F 3 "" H 9100 1300 50  0001 C CNN
+	1    9100 1300
+	1    0    0    -1
+$EndComp
+Wire Wire Line
+	9100 1200 9100 1300
+Wire Wire Line
+	9100 800  9100 900
 $EndSCHEMATC

Commit message: Updated PCB and code
Parts:
- removed unit 1 of U4
- added C3, C4, C6, C7: 1uF, Capacitor_SMD:C_1206_3216Metric, symbol Device:C
- added U4: OPA277, Package_SON:Texas_S-PVSON-N8, symbol Amplifier_Operational:LM741
- U5: renamed from U4; footprint Package_SON:Texas_S-PVSON-N8 -> (none)
- renumbered C3 to C5, J3 to J1, J1 to J2, J4 to J3, J5 to J4, J2 to J5, R7 to R3, R6 to R4, R3 to R5, R4 to R6, R5 to R7, U5 to U6
Connections:
- net labels added: A, B, Load_In, MOSFET_Drain
- wire segments 112 -> 127
- no-connect marks 1 -> 3

Commit message: Updated PCB
Added potentiometers instead of fixed resistors on R6 and R7. Allows accurate changing of resistance to get good current ranges
Parts:
- removed R6, R7: R, Resistor_SMD:R_1206_3216Metric, symbol Device:R
- removed U5: OPA2277, symbol Amplifier_Operational:OPA2277
- added RV1, RV2: R_POT, Potentiometer_THT:Potentiometer_Bourns_3266Y_Vertical, symbol Device:R_POT
Connections:
- wire segments 127 -> 129
Changed lines of the file:
@@
 Text Notes 6300 2650 0    50   ~ 0
 26.7mV/A
-$Comp
-L Amplifier_Operational:OPA2277 U5
-U 3 1 61101BF2
-P 6450 7050
-F 0 "U5" H 6408 7096 50  0000 L CNN
-F 1 "OPA2277" H 6408 7005 50  0000 L CNN
-F 2 "" H 6450 7050 50  0001 C CNN
-F 3 "https://www.ti.com/lit/ds/symlink/opa2277.pdf" H 6450 7050 50  0001 C CNN
-	3    6450 7050
-	1    0    0    -1
-$EndComp
-$Comp
-L power:+5V #PWR020
-U 1 1 61108070
-P 6350 6650
-F 0 "#PWR020" H 6350 6500 50  0001 C CNN
-F 1 "+5V" H 6365 6823 50  0000 C CNN
-F 2 "" H 6350 6650 50  0001 C CNN
-F 3 "" H 6350 6650 50  0001 C CNN
-	1    6350 6650
-	1    0    0    -1
-$EndComp
-$Comp
-L power:GND #PWR021
-U 1 1 61108537
-P 6350 7450
-F 0 "#PWR021" H 6350 7200 50  0001 C CNN
-F 1 "GND" H 6355 7277 50  0000 C CNN
-F 2 "" H 6350 7450 50  0001 C CNN
-F 3 "" H 6350 7450 50  0001 C CNN
-	1    6350 7450
-	1    0    0    -1
-$EndComp
-Wire Wire Line
-	6350 6650 6350 6750
-Wire Wire Line
-	6350 7350 6350 7450
 Text Notes 6350 2900 0    50   ~ 0
 0.6V Min
@@
 L power:+5V #PWR016
 U 1 1 6111B03E
-P 4600 2350
-F 0 "#PWR016" H 4600 2200 50  0001 C CNN
-F 1 "+5V" H 4615 2523 50  0000 C CNN
-F 2 "" H 4600 2350 50  0001 C CNN
-F 3 "" H 4600 2350 50  0001 C CNN
-	1    4600 2350
+P 4700 2300
+F 0 "#PWR016" H 4700 2150 50  0001 C CNN
+F 1 "+5V" H 4715 2473 50  0000 C CNN
+F 2 "" H 4700 2300 50  0001 C CNN
+F 3 "" H 4700 2300 50  0001 C CNN
+	1    4700 2300
 	1    0    0    -1
 $EndComp
@@
 Wire Wire Line
 	5750 3550 7150 3550
-$Comp
-L Device:R R6
-U 1 1 61131D4B
-P 4600 2550
-F 0 "R6" H 4670 2596 50  0000 L CNN
-F 1 "R" H 4670 2505 50  0000 L CNN
-F 2 "Resistor_SMD:R_1206_3216Metric" V 4530 2550 50  0001 C CNN
-F 3 "~" H 4600 2550 50  0001 C CNN
-	1    4600 2550
-	1    0    0    -1
-$EndComp
-$Comp
-L Device:R R7
-U 1 1 61132207
-P 4600 3150
-F 0 "R7" H 4670 3196 50  0000 L CNN
-F 1 "R" H 4670 3105 50  0000 L CNN
-F 2 "Resistor_SMD:R_1206_3216Metric" V 4530 3150 50  0001 C CNN
-F 3 "~" H 4600 3150 50  0001 C CNN
-	1    4600 3150
-	1    0    0    -1
-$EndComp
 $Comp
 L Electronic~Load:MCP4551 U2
@@
 $EndComp
 Wire Wire Line
-	4600 2350 4600 2400
-Wire Wire Line
-	4600 2700 4300 2700
-Wire Wire Line
-	4300 3000 4600 3000
+	4700 2300 4700 2350
 Wire Wire Line
 	4600 3300 4600 3350
@@
 	1950 2150 2050 2150
 NoConn ~ 1950 1350
+$Comp
+L Device:R_POT RV2
+U 1 1 611EDD64
+P 4700 2500
+F 0 "RV2" H 4630 2454 50  0000 R CNN
+F 1 "R_POT" H 4630 2545 50  0000 R CNN
+F 2 "Potentiometer_THT:Potentiometer_Bourns_3266Y_Vertical" H 4700 2500 50  0001 C CNN
+F 3 "~" H 4700 2500 50  0001 C CNN
+	1    4700 2500
+	-1   0    0    1
+$EndComp
+Wire Wire Line
+	4550 2500 4450 2500
+Wire Wire Line
+	4450 2500 4450 2700
+Wire Wire Line
+	4450 2700 4300 2700
+$Comp
+L Device:R_POT RV1
+U 1 1 611F7F26
+P 4600 3150
+F 0 "RV1" H 4530 3104 50  0000 R CNN
+F 1 "R_POT" H 4530 3195 50  0000 R CNN
+F 2 "Potentiometer_THT:Potentiometer_Bourns_3266Y_Vertical" H 4600 3150 50  0001 C CNN
+F 3 "~" H 4600 3150 50  0001 C CNN
+	1    4600 3150
+	-1   0    0    1
+$EndComp
+Wire Wire Line
+	4300 3000 4400 3000
+Wire Wire Line
+	4400 3000 4400 3150
+Wire Wire Line
+	4400 3150 4450 3150
 $EndSCHEMATC
